File: kicad/placa_receptora/placa_receptora.kicad_sch (KiCad schematic)
At the start: 11 parts

Commit message: wip
Parts:
- added C1: C, symbol Device:C
- added JP1, JP2, JP3, JP4: Jumper_2_Open, Jumper:SolderJumper-2_P1.3mm_Open_RoundedPad1.0x1.5mm, symbol Jumper:Jumper_2_Open
- added Q1, Q2, Q3, Q4, Q5, Q6, Q7, Q8: BC168, Package_TO_SOT_THT:TO-92_Inline, symbol Transistor_BJT:BC548
- added R1, R11, R13, R15, R3, R5, R7, R9: 3,9K, Resistor_THT:R_Axial_DIN0207_L6.3mm_D2.5mm_P10.16mm_Horizontal, symbol Device:R
- added R10, R12, R14, R16, R2, R4, R6, R8: 1k, Resistor_THT:R_Axial_DIN0207_L6.3mm_D2.5mm_P10.16mm_Horizontal, symbol Device:R
- added U1: 74LS04, Package_DIP:DIP-14_W7.62mm_Socket_LongPads, symbol 74xx:74LS04
- added U10: 74LS00, Package_DIP:DIP-14_W7.62mm_Socket_LongPads, symbol 74xx:74LS00
- added U11: 74LS121, Package_DIP:DIP-14_W7.62mm_Socket_LongPads, symbol 74xx:74LS121
- added U12, U13: 74LS195, Package_DIP:DIP-16_W7.62mm_Socket_LongPads, symbol 74xx:74LS195
- added unit 3 of U8
- U2, U6, U8: renamed from U?; footprint (none) -> Package_DIP:DIP-14_W7.62mm_Socket_LongPads
- U3, U7, U9: renamed from U?; footprint (none) -> Package_DIP:DIP-24_W15.24mm_Socket_LongPads
- U4, U5: renamed from U?; footprint (none) -> Package_DIP:DIP-16_W7.62mm_Socket_LongPads
- gave numbers to parts that had none: 1
Connections:
- net +5V: now also U4.1 (~{MR}), U5.1 (~{MR}), C1.1, R10.1, R12.1, R14.1, R16.1, R2.1, R4.1, R6.1, R8.1, U12.1 (~{MR}), U12.16 (VCC), U13.1 (~{MR}), U13.16 (VCC), U8.14 (VCC)
- net D0: now also Q1.1 (C), R2.2
- net D1: now also Q2.1 (C), R4.2
- net D2: now also Q3.1 (C), R6.2
- net D3: now also Q4.1 (C), R8.2
- net D4: now also Q5.1 (C), R10.2
- net D5: now also Q6.1 (C), R12.2
- net D6: now also Q7.1 (C), R14.2
- net D7: now also Q8.1 (C), R16.2
- net GND: now also C1.2, Q1.3 (E), Q2.3 (E), Q3.3 (E), Q4.3 (E), Q5.3 (E), Q6.3 (E), Q7.3 (E), Q8.3 (E), U12.8 (GND), U13.8 (GND), U8.7 (GND)
- net /E: now also U3.19 (E1); no longer U3.18 (E0)
- net /Q5: now also U6.4, U6.5; no longer U6.10, U6.9
- net at U2.4: now also U6.6; no longer U6.8
- net at U2.6: now also U3.18 (E0); no longer U3.19 (E1)
- net at U4.2 (J), U4.3 (~{K}): now also JP1.2 (B), JP2.2 (B), U10.1
- new net: JP2.1 (A), U1.11, U1.4
- new net: R1.1, U12.12 (Q3)
- new net: R3.1, U12.13 (Q2)
- new net: R5.1, U12.14 (Q1)
- new net: R7.1, U12.15 (Q0)
- new net: R9.1, U12.2 (J), U12.3 (~{K}), U13.12 (Q3)
- new net: R13.1, U13.14 (Q1)
- new net: Q7.2 (B), R13.2
- new net: Q6.2 (B), R11.2
- new net: Q8.2 (B), R15.2
- new net: R11.1, U13.13 (Q2)
- new net: JP3.1 (A), U1.8
- new net: JP3.2 (B), JP4.2 (B), U13.2 (J), U13.3 (~{K})
- new net: Q4.2 (B), R7.2
- new net: Q5.2 (B), R9.2
- new net: Q3.2 (B), R5.2
- new net: U10.10, U10.3
- new net: U10.5, U10.8
- new net: U10.6, U10.9
- new net: U10.2, U10.4, U11.1 (~{Q})
- new net: JP1.1 (A), U1.10
- new net: R15.1, U13.15 (Q0)
- new net: Q1.2 (B), R1.2
- new net: JP4.1 (A), U1.6, U1.9
- new net: Q2.2 (B), R3.2
- no-connect marks 10 -> 12
Other:
- moved on the sheet: U2A, U4, U5, U6B

Commit message: mais alguns avanções na PCB da interface receptora
Parts:
- added unit 4 of U10
- added U14, U15, U16: 74LS93, Package_DIP:DIP-14_W7.62mm_Socket_LongPads, symbol 74xx:74LS93
- C1: footprint (none) -> Capacitor_THT:CP_Axial_L11.0mm_D5.0mm_P18.00mm_Horizontal
Connections:
- net +5V: now also U14.5 (VCC), U15.5 (VCC), U16.5 (VCC)
- net GND: now also U14.10 (GND), U15.10 (GND), U16.10 (GND)
- net at U11.3 (A1): now also U11.4 (A2), U10.11
- new net: U10.12, U14.12 (Q0)
- new net: U10.13, U14.9 (Q1)
- new net: U16.11 (Q3), U16.14 (CP0)
- new net: U15.1 (CP1..3), U16.12 (Q0)
- new net: U14.2 (R0(1)), U14.3 (R0(2)), U15.2 (R0(1)), U15.3 (R0(2)), U16.2 (R0(1)), U16.3 (R0(2))
- new net: U14.1 (CP1..3), U15.12 (Q0)
- new net: U14.11 (Q3), U14.14 (CP0)
- new net: U15.11 (Q3), U15.14 (CP0)
- no-connect marks 12 -> 17
Other:
- note added: "Monostable Multivibrator with Schmitt-trigger Inputs"

Commit message: mais um pouco da PCB da placa receptora
Parts:
- added C2: C, Capacitor_THT:CP_Radial_D6.3mm_P2.50mm, symbol Device:C
- added unit 5 of U10
- added unit 3 of U2
- added unit 2 of U8
Connections:
- net +5V: now also U11.14 (VCC), U11.5 (B), U11.9 (Rint), U10.14 (VCC), U2.14 (VCC)
- net GND: now also U11.7 (GND), U10.7 (GND), U2.7 (GND)
- net CLOCK_PULSE: now reaches U12.10 (CP)
- net CLOCK_PULSE: now also U13.10 (CP), U14.1 (CP1..3), U15.12 (Q0), U4.10 (CP), U5.10 (CP)
- net at U11.10 (Cext): now also C2.1
- net at U11.11 (R/Cext): now also C2.2
- net at U11.6 (Q): now also U8.10, U8.12, U8.13, U8.9
Other:
- moved on the sheet: C1, J1, JP1, JP2, JP3, JP4, Q1, Q2, Q3, Q4, Q5, Q6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
